Commit message: r50 v2

File: source/isaaclab_tasks/isaaclab_tasks/manager_based/manipulation/lift/robot_model/arm_description/urdf/R50/r50_v4.urdf (robot description, URDF)
Before this commit: robot 00_r50_arm_2_7_asm_09059.SLDASM, 15 links, 14 joints
Joints:
- joint M3: limit lower=2.72 upper=4.53 effort=0 velocity=0 -> lower=2.72 upper=4.53 effort=100 velocity=5
- joint M4: limit lower=0.87 upper=2.09 effort=0 velocity=0 -> lower=0.87 upper=2.09 effort=100 velocity=5
- joint M5: limit lower=-2.4422 upper=3.1416 effort=0 velocity=0 -> lower=-2.4422 upper=3.1416 effort=100 velocity=5
- joint M6_1: limit lower=0 upper=1.7453 effort=0 velocity=0 -> lower=0 upper=1.7453 effort=100 velocity=5
- joint M6_2: limit lower=0 upper=1.7453 effort=0 velocity=0 -> lower=0 upper=1.7453 effort=100 velocity=5

File: source/isaaclab_tasks/isaaclab_tasks/manager_based/manipulation/lift/robot_model/arm_description/urdf/R50/r50_v5.urdf (robot description, URDF)
Before this commit: robot 00_r50_arm_2_7_asm_09059.SLDASM, 15 links, 14 joints
Links:
- link base_link: geometry collision mesh filename=package://00_r50_arm_2_7_asm_09059.SLDASM/meshes/base_link.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 scale=0.5 0.5 0.5; visual mesh filename=package://00_r50_arm_2_7_asm_09059.SLDASM/meshes/base_link.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 scale=0.5 0.5 0.5
Joints:
- joint M0: limit (none) -> lower=-1.57 upper=1.57 effort=0 velocity=0; type fixed -> continuous
- joint M3: limit lower=3.54 upper=4.7116 effort=1 velocity=1 -> lower=3. upper=5。2 effort=100 velocity=5
- joint M4: limit lower=1.23 upper=3.1416 effort=1 velocity=1 -> lower=1.23 upper=3.1416 effort=100 velocity=5
- joint M5: limit lower=-2.4422 upper=3.1416 effort=1 velocity=1 -> lower=-2.4422 upper=3.1416 effort=100 velocity=5
- joint M6_1: axis 0 0 1 -> 0 1 0; limit lower=0 upper=1.7453 effort=1 velocity=1 -> lower=0.0 upper=0.04 effort=100 velocity=5; type revolute -> prismatic
- joint M6_2: axis 0 0 -1 -> 0 -1 0; limit lower=0 upper=1.7453 effort=1 velocity=1 -> lower=0 upper=0.04 effort=100 velocity=5; type revolute -> prismatic
